Commit message: Fix AGV_Jiont -> AGV_Joint typo everywhere in one commit
joint_state_architecture.md sec 7 required this be decided, not drifted into,
and applied atomically across the URDF and every consumer. 25 occurrences in
11 files.

Functionally this is 5 places that must agree, and a check confirms they now
do (URDF joint definitions, waist_driver.yaml joint_names,
waist_driver_node.py _DEFAULT_JOINTS, joint_state_merger.py WAIST):
  AGV_Joint1, AGV_Joint2

Safer than sec 4.2 assumed, and worth recording why: the typo was confined to
the two <joint name=...> strings in the URDF. The links (AGV_Yaw, AGV_Pitch)
and every mesh file were already spelled correctly, and TF frame ids come from
link names — so no TF frame ever carried the typo and the transform tree is
unchanged by this rename. The neighbouring Left_Joint0 in the same URDF was
already correct, so 'Joint' was the convention all along.

Verified: URDF still parses and yields exactly 29 joints with AGV_Joint1/2 and
untouched AGV_Yaw/AGV_Pitch links; all yaml still loads; every launch file
still compiles and passes the include/argument cross-check.

Remaining exposure is outside this repo: anything that looks these joints up
by NAME rather than by frame (VR teleop, the other machines on this ROS
domain) needs the same rename. Nothing in-repo references them via SRDF,
MoveIt configs or RViz configs — checked.

docs/joint_state_architecture.md sec 4.2 and sec 7 now record the decision and
its rationale instead of still asking for one.

Co-Authored-By: Claude Opus 5 <noreply@anthropic.com>
Claude-Session: https://claude.ai/code/session_01WGZvhU4HjdRHtJvwrwtK47

File: src/flexiv_amr_description/urdf/AICO2-Rizon4.urdf (robot description, URDF)
Before this commit: robot AICO2-Rizon4, 30 links, 29 joints
Joints:
- removed joint AGV_Jiont1
- removed joint AGV_Jiont2
- added joint AGV_Joint1: type revolute, parent base_link, child AGV_Yaw, origin xyz=0 0 0.2975 rpy=0 0 0, axis 0 0 1, limit lower=-1.57 upper=1.57 effort=400 velocity=1
- added joint AGV_Joint2: type revolute, parent AGV_Yaw, child AGV_Pitch, origin xyz=0 0 0 rpy=0 0 0, axis 0 1 0, limit lower=0 upper=1.57 effort=1000 velocity=1

Commit message: URDF: five visual meshes referenced files that have never existed
RViz was drawing an incomplete robot with different links absent on each arm,
and no amount of joint-state or TF work changed it, because the cause is
static: the URDF references mesh files that are not in the package and never
were. `git log --all --diff-filter=ADR` finds no commit that ever added them.

    base_link     meshes/visual/AGV_Base.obj
    AGV_Pitch     meshes/visual/AGV_Pitch.obj
    Left_link2    meshes/visual/link2.obj
    Right_link2   meshes/visual/link2.obj
    Left_link6    meshes/visual/link6.obj

That asymmetry is exactly what was observed: the left arm loses link2 and
link6, the right arm only link2 (Right_link6 uses link6r.obj, which exists).
AGV_Pitch is the link both arms mount to, so the join between body and arms had
no geometry at all and the arms read as wrongly attached.

The giveaway in meshes/visual/ is that link2.mtl and link6.mtl are present
while their .obj geometry is not -- material files survived whatever transfer
lost the meshes.

Each of the five has a collision STL in the same package at an identical
origin, so those references now point at the STLs. Coarser shading, same
geometry, same attachment, and the model is complete from files already
committed. All 52 mesh references now resolve.

If the original .obj files turn up (they are stock Flexiv Rizon and AGV vendor
assets), switching back is a one-line revert of each path.

Co-Authored-By: Claude Opus 5 <noreply@anthropic.com>
Claude-Session: https://claude.ai/code/session_01WGZvhU4HjdRHtJvwrwtK47

File: src/flexiv_amr_description/urdf/AICO2-Rizon4.urdf (robot description, URDF)
Before this commit: robot AICO2-Rizon4, 30 links, 29 joints
Links:
- link AGV_Pitch: geometry collision mesh filename=package://flexiv_amr_description/meshes/collision/AGV_Pitch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; visual mesh filename=package://flexiv_amr_description/meshes/collision/AGV_Pitch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
- link Left_link2: geometry collision mesh filename=package://flexiv_amr_description/meshes/collision/link2.stl; visual mesh filename=package://flexiv_amr_description/meshes/collision/link2.stl
- link Left_link6: geometry collision mesh filename=package://flexiv_amr_description/meshes/collision/link6.stl; visual mesh filename=package://flexiv_amr_description/meshes/collision/link6.stl
- link Right_link2: geometry collision mesh filename=package://flexiv_amr_description/meshes/collision/link2.stl; visual mesh filename=package://flexiv_amr_description/meshes/collision/link2.stl
- link base_link: geometry collision mesh filename=package://flexiv_amr_description/meshes/collision/AGV_Base.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; visual mesh filename=package://flexiv_amr_description/meshes/collision/AGV_Base.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
